File: A3-led-panel/A3-led-panel.kicad_pcb (KiCad board)
At the start: 2 copper layers, 0 parts

Commit message: A3-led-panel: version 1
Parts:
- added +5V: TestPoint_Plated_Hole_D2.0mm, TestPoint:TestPoint_Plated_Hole_D2.0mm, F.Cu at (55.9, 193.0)
- added 1k: R_Axial_DIN0207_L6.3mm_D2.5mm_P10.16mm_Horizontal, Resistor_THT:R_Axial_DIN0207_L6.3mm_D2.5mm_P10.16mm_Horizontal, F.Cu at (421.6, 315.0)
- added 1k: R_Axial_DIN0207_L6.3mm_D2.5mm_P10.16mm_Horizontal, Resistor_THT:R_Axial_DIN0207_L6.3mm_D2.5mm_P10.16mm_Horizontal, F.Cu at (238.8, 315.0)
- added 1k: R_Axial_DIN0207_L6.3mm_D2.5mm_P10.16mm_Horizontal, Resistor_THT:R_Axial_DIN0207_L6.3mm_D2.5mm_P10.16mm_Horizontal, F.Cu at (238.8, 213.4)
- added 1k: R_Axial_DIN0207_L6.3mm_D2.5mm_P10.16mm_Horizontal, Resistor_THT:R_Axial_DIN0207_L6.3mm_D2.5mm_P10.16mm_Horizontal, F.Cu at (218.4, 213.4)
- added 1k: R_Axial_DIN0207_L6.3mm_D2.5mm_P10.16mm_Horizontal, Resistor_THT:R_Axial_DIN0207_L6.3mm_D2.5mm_P10.16mm_Horizontal, F.Cu at (198.1, 213.4)
- added 1k: R_Axial_DIN0207_L6.3mm_D2.5mm_P10.16mm_Horizontal, Resistor_THT:R_Axial_DIN0207_L6.3mm_D2.5mm_P10.16mm_Horizontal, F.Cu at (177.8, 213.4)
- added 1k: R_Axial_DIN0207_L6.3mm_D2.5mm_P10.16mm_Horizontal, Resistor_THT:R_Axial_DIN0207_L6.3mm_D2.5mm_P10.16mm_Horizontal, F.Cu at (157.5, 213.4)
- added 1k: R_Axial_DIN0207_L6.3mm_D2.5mm_P10.16mm_Horizontal, Resistor_THT:R_Axial_DIN0207_L6.3mm_D2.5mm_P10.16mm_Horizontal, F.Cu at (137.2, 213.4)
- added 1k: R_Axial_DIN0207_L6.3mm_D2.5mm_P10.16mm_Horizontal, Resistor_THT:R_Axial_DIN0207_L6.3mm_D2.5mm_P10.16mm_Horizontal, F.Cu at (116.8, 213.4)
- added 1k: R_Axial_DIN0207_L6.3mm_D2.5mm_P10.16mm_Horizontal, Resistor_THT:R_Axial_DIN0207_L6.3mm_D2.5mm_P10.16mm_Horizontal, F.Cu at (96.5, 213.4)
- added 1k: R_Axial_DIN0207_L6.3mm_D2.5mm_P10.16mm_Horizontal, Resistor_THT:R_Axial_DIN0207_L6.3mm_D2.5mm_P10.16mm_Horizontal, F.Cu at (76.2, 213.4)
- added 1k: R_Axial_DIN0207_L6.3mm_D2.5mm_P10.16mm_Horizontal, Resistor_THT:R_Axial_DIN0207_L6.3mm_D2.5mm_P10.16mm_Horizontal, F.Cu at (421.6, 193.0)
- added 1k: R_Axial_DIN0207_L6.3mm_D2.5mm_P10.16mm_Horizontal, Resistor_THT:R_Axial_DIN0207_L6.3mm_D2.5mm_P10.16mm_Horizontal, F.Cu at (218.4, 315.0)
- added 1k: R_Axial_DIN0207_L6.3mm_D2.5mm_P10.16mm_Horizontal, Resistor_THT:R_Axial_DIN0207_L6.3mm_D2.5mm_P10.16mm_Horizontal, F.Cu at (401.3, 193.0)
- added 1k: R_Axial_DIN0207_L6.3mm_D2.5mm_P10.16mm_Horizontal, Resistor_THT:R_Axial_DIN0207_L6.3mm_D2.5mm_P10.16mm_Horizontal, F.Cu at (381.0, 193.0)
- added 1k: R_Axial_DIN0207_L6.3mm_D2.5mm_P10.16mm_Horizontal, Resistor_THT:R_Axial_DIN0207_L6.3mm_D2.5mm_P10.16mm_Horizontal, F.Cu at (360.7, 193.0)
- added 1k: R_Axial_DIN0207_L6.3mm_D2.5mm_P10.16mm_Horizontal, Resistor_THT:R_Axial_DIN0207_L6.3mm_D2.5mm_P10.16mm_Horizontal, F.Cu at (340.4, 193.0)
- added 1k: R_Axial_DIN0207_L6.3mm_D2.5mm_P10.16mm_Horizontal, Resistor_THT:R_Axial_DIN0207_L6.3mm_D2.5mm_P10.16mm_Horizontal, F.Cu at (320.0, 193.0)
- added 1k: R_Axial_DIN0207_L6.3mm_D2.5mm_P10.16mm_Horizontal, Resistor_THT:R_Axial_DIN0207_L6.3mm_D2.5mm_P10.16mm_Horizontal, F.Cu at (299.7, 193.0)
- added 1k: R_Axial_DIN0207_L6.3mm_D2.5mm_P10.16mm_Horizontal, Resistor_THT:R_Axial_DIN0207_L6.3mm_D2.5mm_P10.16mm_Horizontal, F.Cu at (279.4, 193.0)
- added 1k: R_Axial_DIN0207_L6.3mm_D2.5mm_P10.16mm_Horizontal, Resistor_THT:R_Axial_DIN0207_L6.3mm_D2.5mm_P10.16mm_Horizontal, F.Cu at (259.1, 193.0)
- added 1k: R_Axial_DIN0207_L6.3mm_D2.5mm_P10.16mm_Horizontal, Resistor_THT:R_Axial_DIN0207_L6.3mm_D2.5mm_P10.16mm_Horizontal, F.Cu at (238.8, 193.0)
- added 1k: R_Axial_DIN0207_L6.3mm_D2.5mm_P10.16mm_Horizontal, Resistor_THT:R_Axial_DIN0207_L6.3mm_D2.5mm_P10.16mm_Horizontal, F.Cu at (218.4, 193.0)
- added 1k: R_Axial_DIN0207_L6.3mm_D2.5mm_P10.16mm_Horizontal, Resistor_THT:R_Axial_DIN0207_L6.3mm_D2.5mm_P10.16mm_Horizontal, F.Cu at (198.1, 315.0)
- added 1k: R_Axial_DIN0207_L6.3mm_D2.5mm_P10.16mm_Horizontal, Resistor_THT:R_Axial_DIN0207_L6.3mm_D2.5mm_P10.16mm_Horizontal, F.Cu at (198.1, 193.0)
- added 1k: R_Axial_DIN0207_L6.3mm_D2.5mm_P10.16mm_Horizontal, Resistor_THT:R_Axial_DIN0207_L6.3mm_D2.5mm_P10.16mm_Horizontal, F.Cu at (177.8, 193.0)
- added 1k: R_Axial_DIN0207_L6.3mm_D2.5mm_P10.16mm_Horizontal, Resistor_THT:R_Axial_DIN0207_L6.3mm_D2.5mm_P10.16mm_Horizontal, F.Cu at (157.5, 193.0)
- added 1k: R_Axial_DIN0207_L6.3mm_D2.5mm_P10.16mm_Horizontal, Resistor_THT:R_Axial_DIN0207_L6.3mm_D2.5mm_P10.16mm_Horizontal, F.Cu at (137.2, 193.0)
- added 1k: R_Axial_DIN0207_L6.3mm_D2.5mm_P10.16mm_Horizontal, Resistor_THT:R_Axial_DIN0207_L6.3mm_D2.5mm_P10.16mm_Horizontal, F.Cu at (116.8, 193.0)
- added 1k: R_Axial_DIN0207_L6.3mm_D2.5mm_P10.16mm_Horizontal, Resistor_THT:R_Axial_DIN0207_L6.3mm_D2.5mm_P10.16mm_Horizontal, F.Cu at (96.5, 193.0)
- added 1k: R_Axial_DIN0207_L6.3mm_D2.5mm_P10.16mm_Horizontal, Resistor_THT:R_Axial_DIN0207_L6.3mm_D2.5mm_P10.16mm_Horizontal, F.Cu at (76.2, 193.0)
- added 1k: R_Axial_DIN0207_L6.3mm_D2.5mm_P10.16mm_Horizontal, Resistor_THT:R_Axial_DIN0207_L6.3mm_D2.5mm_P10.16mm_Horizontal, F.Cu at (421.6, 172.7)
- added 1k: R_Axial_DIN0207_L6.3mm_D2.5mm_P10.16mm_Horizontal, Resistor_THT:R_Axial_DIN0207_L6.3mm_D2.5mm_P10.16mm_Horizontal, F.Cu at (401.3, 172.7)
- added 1k: R_Axial_DIN0207_L6.3mm_D2.5mm_P10.16mm_Horizontal, Resistor_THT:R_Axial_DIN0207_L6.3mm_D2.5mm_P10.16mm_Horizontal, F.Cu at (381.0, 172.7)
- added 1k: R_Axial_DIN0207_L6.3mm_D2.5mm_P10.16mm_Horizontal, Resistor_THT:R_Axial_DIN0207_L6.3mm_D2.5mm_P10.16mm_Horizontal, F.Cu at (177.8, 315.0)
- added 1k: R_Axial_DIN0207_L6.3mm_D2.5mm_P10.16mm_Horizontal, Resistor_THT:R_Axial_DIN0207_L6.3mm_D2.5mm_P10.16mm_Horizontal, F.Cu at (360.7, 172.7)
- added 1k: R_Axial_DIN0207_L6.3mm_D2.5mm_P10.16mm_Horizontal, Resistor_THT:R_Axial_DIN0207_L6.3mm_D2.5mm_P10.16mm_Horizontal, F.Cu at (340.4, 172.7)
- added 1k: R_Axial_DIN0207_L6.3mm_D2.5mm_P10.16mm_Horizontal, Resistor_THT:R_Axial_DIN0207_L6.3mm_D2.5mm_P10.16mm_Horizontal, F.Cu at (320.0, 172.7)
- added 1k: R_Axial_DIN0207_L6.3mm_D2.5mm_P10.16mm_Horizontal, Resistor_THT:R_Axial_DIN0207_L6.3mm_D2.5mm_P10.16mm_Horizontal, F.Cu at (299.7, 172.7)
- added 1k: R_Axial_DIN0207_L6.3mm_D2.5mm_P10.16mm_Horizontal, Resistor_THT:R_Axial_DIN0207_L6.3mm_D2.5mm_P10.16mm_Horizontal, F.Cu at (279.4, 172.7)
- added 1k: R_Axial_DIN0207_L6.3mm_D2.5mm_P10.16mm_Horizontal, Resistor_THT:R_Axial_DIN0207_L6.3mm_D2.5mm_P10.16mm_Horizontal, F.Cu at (259.1, 172.7)
- added 1k: R_Axial_DIN0207_L6.3mm_D2.5mm_P10.16mm_Horizontal, Resistor_THT:R_Axial_DIN0207_L6.3mm_D2.5mm_P10.16mm_Horizontal, F.Cu at (238.8, 172.7)
- added 1k: R_Axial_DIN0207_L6.3mm_D2.5mm_P10.16mm_Horizontal, Resistor_THT:R_Axial_DIN0207_L6.3mm_D2.5mm_P10.16mm_Horizontal, F.Cu at (218.4, 172.7)
- added 1k: R_Axial_DIN0207_L6.3mm_D2.5mm_P10.16mm_Horizontal, Resistor_THT:R_Axial_DIN0207_L6.3mm_D2.5mm_P10.16mm_Horizontal, F.Cu at (198.1, 172.7)
- added 1k: R_Axial_DIN0207_L6.3mm_D2.5mm_P10.16mm_Horizontal, Resistor_THT:R_Axial_DIN0207_L6.3mm_D2.5mm_P10.16mm_Horizontal, F.Cu at (177.8, 172.7)
- added 1k: R_Axial_DIN0207_L6.3mm_D2.5mm_P10.16mm_Horizontal, Resistor_THT:R_Axial_DIN0207_L6.3mm_D2.5mm_P10.16mm_Horizontal, F.Cu at (157.5, 315.0)
- added 1k: R_Axial_DIN0207_L6.3mm_D2.5mm_P10.16mm_Horizontal, Resistor_THT:R_Axial_DIN0207_L6.3mm_D2.5mm_P10.16mm_Horizontal, F.Cu at (157.5, 172.7)
- added 1k: R_Axial_DIN0207_L6.3mm_D2.5mm_P10.16mm_Horizontal, Resistor_THT:R_Axial_DIN0207_L6.3mm_D2.5mm_P10.16mm_Horizontal, F.Cu at (137.2, 172.7)
- added 1k: R_Axial_DIN0207_L6.3mm_D2.5mm_P10.16mm_Horizontal, Resistor_THT:R_Axial_DIN0207_L6.3mm_D2.5mm_P10.16mm_Horizontal, F.Cu at (116.8, 172.7)
- added 1k: R_Axial_DIN0207_L6.3mm_D2.5mm_P10.16mm_Horizontal, Resistor_THT:R_Axial_DIN0207_L6.3mm_D2.5mm_P10.16mm_Horizontal, F.Cu at (96.5, 172.7)
- added 1k: R_Axial_DIN0207_L6.3mm_D2.5mm_P10.16mm_Horizontal, Resistor_THT:R_Axial_DIN0207_L6.3mm_D2.5mm_P10.16mm_Horizontal, F.Cu at (76.2, 172.7)
- added 1k: R_Axial_DIN0207_L6.3mm_D2.5mm_P10.16mm_Horizontal, Resistor_THT:R_Axial_DIN0207_L6.3mm_D2.5mm_P10.16mm_Horizontal, F.Cu at (421.6, 152.4)
- added 1k: R_Axial_DIN0207_L6.3mm_D2.5mm_P10.16mm_Horizontal, Resistor_THT:R_Axial_DIN0207_L6.3mm_D2.5mm_P10.16mm_Horizontal, F.Cu at (401.3, 152.4)
- added 1k: R_Axial_DIN0207_L6.3mm_D2.5mm_P10.16mm_Horizontal, Resistor_THT:R_Axial_DIN0207_L6.3mm_D2.5mm_P10.16mm_Horizontal, F.Cu at (381.0, 152.4)
- added 1k: R_Axial_DIN0207_L6.3mm_D2.5mm_P10.16mm_Horizontal, Resistor_THT:R_Axial_DIN0207_L6.3mm_D2.5mm_P10.16mm_Horizontal, F.Cu at (360.7, 152.4)
- added 1k: R_Axial_DIN0207_L6.3mm_D2.5mm_P10.16mm_Horizontal, Resistor_THT:R_Axial_DIN0207_L6.3mm_D2.5mm_P10.16mm_Horizontal, F.Cu at (340.4, 152.4)
- added 1k: R_Axial_DIN0207_L6.3mm_D2.5mm_P10.16mm_Horizontal, Resistor_THT:R_Axial_DIN0207_L6.3mm_D2.5mm_P10.16mm_Horizontal, F.Cu at (137.2, 315.0)
- added 1k: R_Axial_DIN0207_L6.3mm_D2.5mm_P10.16mm_Horizontal, Resistor_THT:R_Axial_DIN0207_L6.3mm_D2.5mm_P10.16mm_Horizontal, F.Cu at (320.0, 152.4)
- added 1k: R_Axial_DIN0207_L6.3mm_D2.5mm_P10.16mm_Horizontal, Resistor_THT:R_Axial_DIN0207_L6.3mm_D2.5mm_P10.16mm_Horizontal, F.Cu at (299.7, 152.4)
- added 1k: R_Axial_DIN0207_L6.3mm_D2.5mm_P10.16mm_Horizontal, Resistor_THT:R_Axial_DIN0207_L6.3mm_D2.5mm_P10.16mm_Horizontal, F.Cu at (279.4, 152.4)
- added 1k: R_Axial_DIN0207_L6.3mm_D2.5mm_P10.16mm_Horizontal, Resistor_THT:R_Axial_DIN0207_L6.3mm_D2.5mm_P10.16mm_Horizontal, F.Cu at (259.1, 152.4)
- added 1k: R_Axial_DIN0207_L6.3mm_D2.5mm_P10.16mm_Horizontal, Resistor_THT:R_Axial_DIN0207_L6.3mm_D2.5mm_P10.16mm_Horizontal, F.Cu at (238.8, 152.4)
- added 1k: R_Axial_DIN0207_L6.3mm_D2.5mm_P10.16mm_Horizontal, Resistor_THT:R_Axial_DIN0207_L6.3mm_D2.5mm_P10.16mm_Horizontal, F.Cu at (218.4, 152.4)
- added 1k: R_Axial_DIN0207_L6.3mm_D2.5mm_P10.16mm_Horizontal, Resistor_THT:R_Axial_DIN0207_L6.3mm_D2.5mm_P10.16mm_Horizontal, F.Cu at (198.1, 152.4)
- added 1k: R_Axial_DIN0207_L6.3mm_D2.5mm_P10.16mm_Horizontal, Resistor_THT:R_Axial_DIN0207_L6.3mm_D2.5mm_P10.16mm_Horizontal, F.Cu at (177.8, 152.4)
- added 1k: R_Axial_DIN0207_L6.3mm_D2.5mm_P10.16mm_Horizontal, Resistor_THT:R_Axial_DIN0207_L6.3mm_D2.5mm_P10.16mm_Horizontal, F.Cu at (157.5, 152.4)
- added 1k: R_Axial_DIN0207_L6.3mm_D2.5mm_P10.16mm_Horizontal, Resistor_THT:R_Axial_DIN0207_L6.3mm_D2.5mm_P10.16mm_Horizontal, F.Cu at (137.2, 152.4)
- added 1k: R_Axial_DIN0207_L6.3mm_D2.5mm_P10.16mm_Horizontal, Resistor_THT:R_Axial_DIN0207_L6.3mm_D2.5mm_P10.16mm_Horizontal, F.Cu at (116.8, 315.0)
- added 1k: R_Axial_DIN0207_L6.3mm_D2.5mm_P10.16mm_Horizontal, Resistor_THT:R_Axial_DIN0207_L6.3mm_D2.5mm_P10.16mm_Horizontal, F.Cu at (116.8, 152.4)
- added 1k: R_Axial_DIN0207_L6.3mm_D2.5mm_P10.16mm_Horizontal, Resistor_THT:R_Axial_DIN0207_L6.3mm_D2.5mm_P10.16mm_Horizontal, F.Cu at (96.5, 152.4)
- added 1k: R_Axial_DIN0207_L6.3mm_D2.5mm_P10.16mm_Horizontal, Resistor_THT:R_Axial_DIN0207_L6.3mm_D2.5mm_P10.16mm_Horizontal, F.Cu at (76.2, 152.4)
- added 1k: R_Axial_DIN0207_L6.3mm_D2.5mm_P10.16mm_Horizontal, Resistor_THT:R_Axial_DIN0207_L6.3mm_D2.5mm_P10.16mm_Horizontal, F.Cu at (421.6, 132.1)
- added 1k: R_Axial_DIN0207_L6.3mm_D2.5mm_P10.16mm_Horizontal, Resistor_THT:R_Axial_DIN0207_L6.3mm_D2.5mm_P10.16mm_Horizontal, F.Cu at (401.3, 132.1)
- added 1k: R_Axial_DIN0207_L6.3mm_D2.5mm_P10.16mm_Horizontal, Resistor_THT:R_Axial_DIN0207_L6.3mm_D2.5mm_P10.16mm_Horizontal, F.Cu at (381.0, 132.1)
- added 1k: R_Axial_DIN0207_L6.3mm_D2.5mm_P10.16mm_Horizontal, Resistor_THT:R_Axial_DIN0207_L6.3mm_D2.5mm_P10.16mm_Horizontal, F.Cu at (360.7, 132.1)
- added 1k: R_Axial_DIN0207_L6.3mm_D2.5mm_P10.16mm_Horizontal, Resistor_THT:R_Axial_DIN0207_L6.3mm_D2.5mm_P10.16mm_Horizontal, F.Cu at (340.4, 132.1)
- added 1k: R_Axial_DIN0207_L6.3mm_D2.5mm_P10.16mm_Horizontal, Resistor_THT:R_Axial_DIN0207_L6.3mm_D2.5mm_P10.16mm_Horizontal, F.Cu at (320.0, 132.1)
- added 1k: R_Axial_DIN0207_L6.3mm_D2.5mm_P10.16mm_Horizontal, Resistor_THT:R_Axial_DIN0207_L6.3mm_D2.5mm_P10.16mm_Horizontal, F.Cu at (299.7, 132.1)
- added 1k: R_Axial_DIN0207_L6.3mm_D2.5mm_P10.16mm_Horizontal, Resistor_THT:R_Axial_DIN0207_L6.3mm_D2.5mm_P10.16mm_Horizontal, F.Cu at (96.5, 315.0)
- added 1k: R_Axial_DIN0207_L6.3mm_D2.5mm_P10.16mm_Horizontal, Resistor_THT:R_Axial_DIN0207_L6.3mm_D2.5mm_P10.16mm_Horizontal, F.Cu at (279.4, 132.1)
- added 1k: R_Axial_DIN0207_L6.3mm_D2.5mm_P10.16mm_Horizontal, Resistor_THT:R_Axial_DIN0207_L6.3mm_D2.5mm_P10.16mm_Horizontal, F.Cu at (259.1, 132.1)
- added 1k: R_Axial_DIN0207_L6.3mm_D2.5mm_P10.16mm_Horizontal, Resistor_THT:R_Axial_DIN0207_L6.3mm_D2.5mm_P10.16mm_Horizontal, F.Cu at (238.8, 132.1)
- added 1k: R_Axial_DIN0207_L6.3mm_D2.5mm_P10.16mm_Horizontal, Resistor_THT:R_Axial_DIN0207_L6.3mm_D2.5mm_P10.16mm_Horizontal, F.Cu at (218.4, 132.1)
- added 1k: R_Axial_DIN0207_L6.3mm_D2.5mm_P10.16mm_Horizontal, Resistor_THT:R_Axial_DIN0207_L6.3mm_D2.5mm_P10.16mm_Horizontal, F.Cu at (198.1, 132.1)
- added 1k: R_Axial_DIN0207_L6.3mm_D2.5mm_P10.16mm_Horizontal, Resistor_THT:R_Axial_DIN0207_L6.3mm_D2.5mm_P10.16mm_Horizontal, F.Cu at (177.8, 132.1)
- added 1k: R_Axial_DIN0207_L6.3mm_D2.5mm_P10.16mm_Horizontal, Resistor_THT:R_Axial_DIN0207_L6.3mm_D2.5mm_P10.16mm_Horizontal, F.Cu at (157.5, 132.1)
- added 1k: R_Axial_DIN0207_L6.3mm_D2.5mm_P10.16mm_Horizontal, Resistor_THT:R_Axial_DIN0207_L6.3mm_D2.5mm_P10.16mm_Horizontal, F.Cu at (137.2, 132.1)
- added 1k: R_Axial_DIN0207_L6.3mm_D2.5mm_P10.16mm_Horizontal, Resistor_THT:R_Axial_DIN0207_L6.3mm_D2.5mm_P10.16mm_Horizontal, F.Cu at (116.8, 132.1)
- added 1k: R_Axial_DIN0207_L6.3mm_D2.5mm_P10.16mm_Horizontal, Resistor_THT:R_Axial_DIN0207_L6.3mm_D2.5mm_P10.16mm_Horizontal, F.Cu at (96.5, 132.1)
- added 1k: R_Axial_DIN0207_L6.3mm_D2.5mm_P10.16mm_Horizontal, Resistor_THT:R_Axial_DIN0207_L6.3mm_D2.5mm_P10.16mm_Horizontal, F.Cu at (76.2, 315.0)
- added 1k: R_Axial_DIN0207_L6.3mm_D2.5mm_P10.16mm_Horizontal, Resistor_THT:R_Axial_DIN0207_L6.3mm_D2.5mm_P10.16mm_Horizontal, F.Cu at (76.2, 132.1)
- added 1k: R_Axial_DIN0207_L6.3mm_D2.5mm_P10.16mm_Horizontal, Resistor_THT:R_Axial_DIN0207_L6.3mm_D2.5mm_P10.16mm_Horizontal, F.Cu at (421.6, 111.8)
- added 1k: R_Axial_DIN0207_L6.3mm_D2.5mm_P10.16mm_Horizontal, Resistor_THT:R_Axial_DIN0207_L6.3mm_D2.5mm_P10.16mm_Horizontal, F.Cu at (401.3, 111.8)
- added 1k: R_Axial_DIN0207_L6.3mm_D2.5mm_P10.16mm_Horizontal, Resistor_THT:R_Axial_DIN0207_L6.3mm_D2.5mm_P10.16mm_Horizontal, F.Cu at (381.0, 111.8)
- added 1k: R_Axial_DIN0207_L6.3mm_D2.5mm_P10.16mm_Horizontal, Resistor_THT:R_Axial_DIN0207_L6.3mm_D2.5mm_P10.16mm_Horizontal, F.Cu at (360.7, 111.8)
- added 1k: R_Axial_DIN0207_L6.3mm_D2.5mm_P10.16mm_Horizontal, Resistor_THT:R_Axial_DIN0207_L6.3mm_D2.5mm_P10.16mm_Horizontal, F.Cu at (340.4, 111.8)
- added 1k: R_Axial_DIN0207_L6.3mm_D2.5mm_P10.16mm_Horizontal, Resistor_THT:R_Axial_DIN0207_L6.3mm_D2.5mm_P10.16mm_Horizontal, F.Cu at (320.0, 111.8)
- added 1k: R_Axial_DIN0207_L6.3mm_D2.5mm_P10.16mm_Horizontal, Resistor_THT:R_Axial_DIN0207_L6.3mm_D2.5mm_P10.16mm_Horizontal, F.Cu at (299.7, 111.8)
- added 1k: R_Axial_DIN0207_L6.3mm_D2.5mm_P10.16mm_Horizontal, Resistor_THT:R_Axial_DIN0207_L6.3mm_D2.5mm_P10.16mm_Horizontal, F.Cu at (279.4, 111.8)
- added 1k: R_Axial_DIN0207_L6.3mm_D2.5mm_P10.16mm_Horizontal, Resistor_THT:R_Axial_DIN0207_L6.3mm_D2.5mm_P10.16mm_Horizontal, F.Cu at (259.1, 111.8)
- added 1k: R_Axial_DIN0207_L6.3mm_D2.5mm_P10.16mm_Horizontal, Resistor_THT:R_Axial_DIN0207_L6.3mm_D2.5mm_P10.16mm_Horizontal, F.Cu at (421.6, 294.6)
- added 1k: R_Axial_DIN0207_L6.3mm_D2.5mm_P10.16mm_Horizontal, Resistor_THT:R_Axial_DIN0207_L6.3mm_D2.5mm_P10.16mm_Horizontal, F.Cu at (238.8, 111.8)
- added 1k: R_Axial_DIN0207_L6.3mm_D2.5mm_P10.16mm_Horizontal, Resistor_THT:R_Axial_DIN0207_L6.3mm_D2.5mm_P10.16mm_Horizontal, F.Cu at (218.4, 111.8)
- added 1k: R_Axial_DIN0207_L6.3mm_D2.5mm_P10.16mm_Horizontal, Resistor_THT:R_Axial_DIN0207_L6.3mm_D2.5mm_P10.16mm_Horizontal, F.Cu at (198.1, 111.8)
- added 1k: R_Axial_DIN0207_L6.3mm_D2.5mm_P10.16mm_Horizontal, Resistor_THT:R_Axial_DIN0207_L6.3mm_D2.5mm_P10.16mm_Horizontal, F.Cu at (177.8, 111.8)
- added 1k: R_Axial_DIN0207_L6.3mm_D2.5mm_P10.16mm_Horizontal, Resistor_THT:R_Axial_DIN0207_L6.3mm_D2.5mm_P10.16mm_Horizontal, F.Cu at (157.5, 111.8)
- added 1k: R_Axial_DIN0207_L6.3mm_D2.5mm_P10.16mm_Horizontal, Resistor_THT:R_Axial_DIN0207_L6.3mm_D2.5mm_P10.16mm_Horizontal, F.Cu at (137.2, 111.8)
- added 1k: R_Axial_DIN0207_L6.3mm_D2.5mm_P10.16mm_Horizontal, Resistor_THT:R_Axial_DIN0207_L6.3mm_D2.5mm_P10.16mm_Horizontal, F.Cu at (116.8, 111.8)
- added 1k: R_Axial_DIN0207_L6.3mm_D2.5mm_P10.16mm_Horizontal, Resistor_THT:R_Axial_DIN0207_L6.3mm_D2.5mm_P10.16mm_Horizontal, F.Cu at (96.5, 111.8)
- added 1k: R_Axial_DIN0207_L6.3mm_D2.5mm_P10.16mm_Horizontal, Resistor_THT:R_Axial_DIN0207_L6.3mm_D2.5mm_P10.16mm_Horizontal, F.Cu at (76.2, 111.8)
- added 1k: R_Axial_DIN0207_L6.3mm_D2.5mm_P10.16mm_Horizontal, Resistor_THT:R_Axial_DIN0207_L6.3mm_D2.5mm_P10.16mm_Horizontal, F.Cu at (421.6, 91.4)
- added 1k: R_Axial_DIN0207_L6.3mm_D2.5mm_P10.16mm_Horizontal, Resistor_THT:R_Axial_DIN0207_L6.3mm_D2.5mm_P10.16mm_Horizontal, F.Cu at (401.3, 315.0)
- added 1k: R_Axial_DIN0207_L6.3mm_D2.5mm_P10.16mm_Horizontal, Resistor_THT:R_Axial_DIN0207_L6.3mm_D2.5mm_P10.16mm_Horizontal, F.Cu at (401.3, 294.6)
- added 1k: R_Axial_DIN0207_L6.3mm_D2.5mm_P10.16mm_Horizontal, Resistor_THT:R_Axial_DIN0207_L6.3mm_D2.5mm_P10.16mm_Horizontal, F.Cu at (401.3, 91.4)
- added 1k: R_Axial_DIN0207_L6.3mm_D2.5mm_P10.16mm_Horizontal, Resistor_THT:R_Axial_DIN0207_L6.3mm_D2.5mm_P10.16mm_Horizontal, F.Cu at (381.0, 91.4)
- added 1k: R_Axial_DIN0207_L6.3mm_D2.5mm_P10.16mm_Horizontal, Resistor_THT:R_Axial_DIN0207_L6.3mm_D2.5mm_P10.16mm_Horizontal, F.Cu at (360.7, 91.4)
- added 1k: R_Axial_DIN0207_L6.3mm_D2.5mm_P10.16mm_Horizontal, Resistor_THT:R_Axial_DIN0207_L6.3mm_D2.5mm_P10.16mm_Horizontal, F.Cu at (340.4, 91.4)
- added 1k: R_Axial_DIN0207_L6.3mm_D2.5mm_P10.16mm_Horizontal, Resistor_THT:R_Axial_DIN0207_L6.3mm_D2.5mm_P10.16mm_Horizontal, F.Cu at (320.0, 91.4)
- added 1k: R_Axial_DIN0207_L6.3mm_D2.5mm_P10.16mm_Horizontal, Resistor_THT:R_Axial_DIN0207_L6.3mm_D2.5mm_P10.16mm_Horizontal, F.Cu at (299.7, 91.4)
- added 1k: R_Axial_DIN0207_L6.3mm_D2.5mm_P10.16mm_Horizontal, Resistor_THT:R_Axial_DIN0207_L6.3mm_D2.5mm_P10.16mm_Horizontal, F.Cu at (279.4, 91.4)
- added 1k: R_Axial_DIN0207_L6.3mm_D2.5mm_P10.16mm_Horizontal, Resistor_THT:R_Axial_DIN0207_L6.3mm_D2.5mm_P10.16mm_Horizontal, F.Cu at (259.1, 91.4)
- added 1k: R_Axial_DIN0207_L6.3mm_D2.5mm_P10.16mm_Horizontal, Resistor_THT:R_Axial_DIN0207_L6.3mm_D2.5mm_P10.16mm_Horizontal, F.Cu at (238.8, 91.4)
- added 1k: R_Axial_DIN0207_L6.3mm_D2.5mm_P10.16mm_Horizontal, Resistor_THT:R_Axial_DIN0207_L6.3mm_D2.5mm_P10.16mm_Horizontal, F.Cu at (218.4, 91.4)
- added 1k: R_Axial_DIN0207_L6.3mm_D2.5mm_P10.16mm_Horizontal, Resistor_THT:R_Axial_DIN0207_L6.3mm_D2.5mm_P10.16mm_Horizontal, F.Cu at (381.0, 294.6)
- added 1k: R_Axial_DIN0207_L6.3mm_D2.5mm_P10.16mm_Horizontal, Resistor_THT:R_Axial_DIN0207_L6.3mm_D2.5mm_P10.16mm_Horizontal, F.Cu at (198.1, 91.4)
- added 1k: R_Axial_DIN0207_L6.3mm_D2.5mm_P10.16mm_Horizontal, Resistor_THT:R_Axial_DIN0207_L6.3mm_D2.5mm_P10.16mm_Horizontal, F.Cu at (177.8, 91.4)
- added 1k: R_Axial_DIN0207_L6.3mm_D2.5mm_P10.16mm_Horizontal, Resistor_THT:R_Axial_DIN0207_L6.3mm_D2.5mm_P10.16mm_Horizontal, F.Cu at (157.5, 91.4)
- added 1k: R_Axial_DIN0207_L6.3mm_D2.5mm_P10.16mm_Horizontal, Resistor_THT:R_Axial_DIN0207_L6.3mm_D2.5mm_P10.16mm_Horizontal, F.Cu at (137.2, 91.4)
- added 1k: R_Axial_DIN0207_L6.3mm_D2.5mm_P10.16mm_Horizontal, Resistor_THT:R_Axial_DIN0207_L6.3mm_D2.5mm_P10.16mm_Horizontal, F.Cu at (116.8, 91.4)
- added 1k: R_Axial_DIN0207_L6.3mm_D2.5mm_P10.16mm_Horizontal, Resistor_THT:R_Axial_DIN0207_L6.3mm_D2.5mm_P10.16mm_Horizontal, F.Cu at (96.5, 91.4)
- added 1k: R_Axial_DIN0207_L6.3mm_D2.5mm_P10.16mm_Horizontal, Resistor_THT:R_Axial_DIN0207_L6.3mm_D2.5mm_P10.16mm_Horizontal, F.Cu at (76.2, 91.4)
- added 1k: R_Axial_DIN0207_L6.3mm_D2.5mm_P10.16mm_Horizontal, Resistor_THT:R_Axial_DIN0207_L6.3mm_D2.5mm_P10.16mm_Horizontal, F.Cu at (421.6, 71.1)
- added 1k: R_Axial_DIN0207_L6.3mm_D2.5mm_P10.16mm_Horizontal, Resistor_THT:R_Axial_DIN0207_L6.3mm_D2.5mm_P10.16mm_Horizontal, F.Cu at (401.3, 71.1)
- added 1k: R_Axial_DIN0207_L6.3mm_D2.5mm_P10.16mm_Horizontal, Resistor_THT:R_Axial_DIN0207_L6.3mm_D2.5mm_P10.16mm_Horizontal, F.Cu at (381.0, 71.1)
- added 1k: R_Axial_DIN0207_L6.3mm_D2.5mm_P10.16mm_Horizontal, Resistor_THT:R_Axial_DIN0207_L6.3mm_D2.5mm_P10.16mm_Horizontal, F.Cu at (360.7, 294.6)
- added 1k: R_Axial_DIN0207_L6.3mm_D2.5mm_P10.16mm_Horizontal, Resistor_THT:R_Axial_DIN0207_L6.3mm_D2.5mm_P10.16mm_Horizontal, F.Cu at (360.7, 71.1)
- added 1k: R_Axial_DIN0207_L6.3mm_D2.5mm_P10.16mm_Horizontal, Resistor_THT:R_Axial_DIN0207_L6.3mm_D2.5mm_P10.16mm_Horizontal, F.Cu at (340.4, 71.1)
- added 1k: R_Axial_DIN0207_L6.3mm_D2.5mm_P10.16mm_Horizontal, Resistor_THT:R_Axial_DIN0207_L6.3mm_D2.5mm_P10.16mm_Horizontal, F.Cu at (320.0, 71.1)
- added 1k: R_Axial_DIN0207_L6.3mm_D2.5mm_P10.16mm_Horizontal, Resistor_THT:R_Axial_DIN0207_L6.3mm_D2.5mm_P10.16mm_Horizontal, F.Cu at (299.7, 71.1)
- added 1k: R_Axial_DIN0207_L6.3mm_D2.5mm_P10.16mm_Horizontal, Resistor_THT:R_Axial_DIN0207_L6.3mm_D2.5mm_P10.16mm_Horizontal, F.Cu at (279.4, 71.1)
- added 1k: R_Axial_DIN0207_L6.3mm_D2.5mm_P10.16mm_Horizontal, Resistor_THT:R_Axial_DIN0207_L6.3mm_D2.5mm_P10.16mm_Horizontal, F.Cu at (259.1, 71.1)
- added 1k: R_Axial_DIN0207_L6.3mm_D2.5mm_P10.16mm_Horizontal, Resistor_THT:R_Axial_DIN0207_L6.3mm_D2.5mm_P10.16mm_Horizontal, F.Cu at (238.8, 71.1)
- added 1k: R_Axial_DIN0207_L6.3mm_D2.5mm_P10.16mm_Horizontal, Resistor_THT:R_Axial_DIN0207_L6.3mm_D2.5mm_P10.16mm_Horizontal, F.Cu at (218.4, 71.1)
- added 1k: R_Axial_DIN0207_L6.3mm_D2.5mm_P10.16mm_Horizontal, Resistor_THT:R_Axial_DIN0207_L6.3mm_D2.5mm_P10.16mm_Horizontal, F.Cu at (198.1, 71.1)
- added 1k: R_Axial_DIN0207_L6.3mm_D2.5mm_P10.16mm_Horizontal, Resistor_THT:R_Axial_DIN0207_L6.3mm_D2.5mm_P10.16mm_Horizontal, F.Cu at (177.8, 71.1)
- added 1k: R_Axial_DIN0207_L6.3mm_D2.5mm_P10.16mm_Horizontal, Resistor_THT:R_Axial_DIN0207_L6.3mm_D2.5mm_P10.16mm_Horizontal, F.Cu at (340.4, 294.6)
- added 1k: R_Axial_DIN0207_L6.3mm_D2.5mm_P10.16mm_Horizontal, Resistor_THT:R_Axial_DIN0207_L6.3mm_D2.5mm_P10.16mm_Horizontal, F.Cu at (157.5, 71.1)
- added 1k: R_Axial_DIN0207_L6.3mm_D2.5mm_P10.16mm_Horizontal, Resistor_THT:R_Axial_DIN0207_L6.3mm_D2.5mm_P10.16mm_Horizontal, F.Cu at (137.2, 71.1)
- added 1k: R_Axial_DIN0207_L6.3mm_D2.5mm_P10.16mm_Horizontal, Resistor_THT:R_Axial_DIN0207_L6.3mm_D2.5mm_P10.16mm_Horizontal, F.Cu at (116.8, 71.1)
- added 1k: R_Axial_DIN0207_L6.3mm_D2.5mm_P10.16mm_Horizontal, Resistor_THT:R_Axial_DIN0207_L6.3mm_D2.5mm_P10.16mm_Horizontal, F.Cu at (96.5, 71.1)
- added 1k: R_Axial_DIN0207_L6.3mm_D2.5mm_P10.16mm_Horizontal, Resistor_THT:R_Axial_DIN0207_L6.3mm_D2.5mm_P10.16mm_Horizontal, F.Cu at (76.2, 71.1)
- added 1k: R_Axial_DIN0207_L6.3mm_D2.5mm_P10.16mm_Horizontal, Resistor_THT:R_Axial_DIN0207_L6.3mm_D2.5mm_P10.16mm_Horizontal, F.Cu at (320.0, 294.6)
- added 1k: R_Axial_DIN0207_L6.3mm_D2.5mm_P10.16mm_Horizontal, Resistor_THT:R_Axial_DIN0207_L6.3mm_D2.5mm_P10.16mm_Horizontal, F.Cu at (299.7, 294.6)
- added 1k: R_Axial_DIN0207_L6.3mm_D2.5mm_P10.16mm_Horizontal, Resistor_THT:R_Axial_DIN0207_L6.3mm_D2.5mm_P10.16mm_Horizontal, F.Cu at (279.4, 294.6)
- added 1k: R_Axial_DIN0207_L6.3mm_D2.5mm_P10.16mm_Horizontal, Resistor_THT:R_Axial_DIN0207_L6.3mm_D2.5mm_P10.16mm_Horizontal, F.Cu at (259.1, 294.6)
- added 1k: R_Axial_DIN0207_L6.3mm_D2.5mm_P10.16mm_Horizontal, Resistor_THT:R_Axial_DIN0207_L6.3mm_D2.5mm_P10.16mm_Horizontal, F.Cu at (238.8, 294.6)
- added 1k: R_Axial_DIN0207_L6.3mm_D2.5mm_P10.16mm_Horizontal, Resistor_THT:R_Axial_DIN0207_L6.3mm_D2.5mm_P10.16mm_Horizontal, F.Cu at (218.4, 294.6)
- added 1k: R_Axial_DIN0207_L6.3mm_D2.5mm_P10.16mm_Horizontal, Resistor_THT:R_Axial_DIN0207_L6.3mm_D2.5mm_P10.16mm_Horizontal, F.Cu at (381.0, 315.0)
- added 1k: R_Axial_DIN0207_L6.3mm_D2.5mm_P10.16mm_Horizontal, Resistor_THT:R_Axial_DIN0207_L6.3mm_D2.5mm_P10.16mm_Horizontal, F.Cu at (198.1, 294.6)
- added 1k: R_Axial_DIN0207_L6.3mm_D2.5mm_P10.16mm_Horizontal, Resistor_THT:R_Axial_DIN0207_L6.3mm_D2.5mm_P10.16mm_Horizontal, F.Cu at (177.8, 294.6)
- added 1k: R_Axial_DIN0207_L6.3mm_D2.5mm_P10.16mm_Horizontal, Resistor_THT:R_Axial_DIN0207_L6.3mm_D2.5mm_P10.16mm_Horizontal, F.Cu at (157.5, 294.6)
- added 1k: R_Axial_DIN0207_L6.3mm_D2.5mm_P10.16mm_Horizontal, Resistor_THT:R_Axial_DIN0207_L6.3mm_D2.5mm_P10.16mm_Horizontal, F.Cu at (137.2, 294.6)
- added 1k: R_Axial_DIN0207_L6.3mm_D2.5mm_P10.16mm_Horizontal, Resistor_THT:R_Axial_DIN0207_L6.3mm_D2.5mm_P10.16mm_Horizontal, F.Cu at (116.8, 294.6)
- added 1k: R_Axial_DIN0207_L6.3mm_D2.5mm_P10.16mm_Horizontal, Resistor_THT:R_Axial_DIN0207_L6.3mm_D2.5mm_P10.16mm_Horizontal, F.Cu at (96.5, 294.6)
- added 1k: R_Axial_DIN0207_L6.3mm_D2.5mm_P10.16mm_Horizontal, Resistor_THT:R_Axial_DIN0207_L6.3mm_D2.5mm_P10.16mm_Horizontal, F.Cu at (76.2, 294.6)
- added 1k: R_Axial_DIN0207_L6.3mm_D2.5mm_P10.16mm_Horizontal, Resistor_THT:R_Axial_DIN0207_L6.3mm_D2.5mm_P10.16mm_Horizontal, F.Cu at (421.6, 274.3)
- added 1k: R_Axial_DIN0207_L6.3mm_D2.5mm_P10.16mm_Horizontal, Resistor_THT:R_Axial_DIN0207_L6.3mm_D2.5mm_P10.16mm_Horizontal, F.Cu at (401.3, 274.3)
- added 1k: R_Axial_DIN0207_L6.3mm_D2.5mm_P10.16mm_Horizontal, Resistor_THT:R_Axial_DIN0207_L6.3mm_D2.5mm_P10.16mm_Horizontal, F.Cu at (381.0, 274.3)
- added 1k: R_Axial_DIN0207_L6.3mm_D2.5mm_P10.16mm_Horizontal, Resistor_THT:R_Axial_DIN0207_L6.3mm_D2.5mm_P10.16mm_Horizontal, F.Cu at (360.7, 315.0)
- added 1k: R_Axial_DIN0207_L6.3mm_D2.5mm_P10.16mm_Horizontal, Resistor_THT:R_Axial_DIN0207_L6.3mm_D2.5mm_P10.16mm_Horizontal, F.Cu at (360.7, 274.3)
- added 1k: R_Axial_DIN0207_L6.3mm_D2.5mm_P10.16mm_Horizontal, Resistor_THT:R_Axial_DIN0207_L6.3mm_D2.5mm_P10.16mm_Horizontal, F.Cu at (340.4, 274.3)
- added 1k: R_Axial_DIN0207_L6.3mm_D2.5mm_P10.16mm_Horizontal, Resistor_THT:R_Axial_DIN0207_L6.3mm_D2.5mm_P10.16mm_Horizontal, F.Cu at (320.0, 274.3)
- added 1k: R_Axial_DIN0207_L6.3mm_D2.5mm_P10.16mm_Horizontal, Resistor_THT:R_Axial_DIN0207_L6.3mm_D2.5mm_P10.16mm_Horizontal, F.Cu at (299.7, 274.3)
- added 1k: R_Axial_DIN0207_L6.3mm_D2.5mm_P10.16mm_Horizontal, Resistor_THT:R_Axial_DIN0207_L6.3mm_D2.5mm_P10.16mm_Horizontal, F.Cu at (279.4, 274.3)
- added 1k: R_Axial_DIN0207_L6.3mm_D2.5mm_P10.16mm_Horizontal, Resistor_THT:R_Axial_DIN0207_L6.3mm_D2.5mm_P10.16mm_Horizontal, F.Cu at (259.1, 274.3)
- added 1k: R_Axial_DIN0207_L6.3mm_D2.5mm_P10.16mm_Horizontal, Resistor_THT:R_Axial_DIN0207_L6.3mm_D2.5mm_P10.16mm_Horizontal, F.Cu at (238.8, 274.3)
- added 1k: R_Axial_DIN0207_L6.3mm_D2.5mm_P10.16mm_Horizontal, Resistor_THT:R_Axial_DIN0207_L6.3mm_D2.5mm_P10.16mm_Horizontal, F.Cu at (218.4, 274.3)
- added 1k: R_Axial_DIN0207_L6.3mm_D2.5mm_P10.16mm_Horizontal, Resistor_THT:R_Axial_DIN0207_L6.3mm_D2.5mm_P10.16mm_Horizontal, F.Cu at (198.1, 274.3)
- added 1k: R_Axial_DIN0207_L6.3mm_D2.5mm_P10.16mm_Horizontal, Resistor_THT:R_Axial_DIN0207_L6.3mm_D2.5mm_P10.16mm_Horizontal, F.Cu at (177.8, 274.3)
- added 1k: R_Axial_DIN0207_L6.3mm_D2.5mm_P10.16mm_Horizontal, Resistor_THT:R_Axial_DIN0207_L6.3mm_D2.5mm_P10.16mm_Horizontal, F.Cu at (340.4, 315.0)
- added 1k: R_Axial_DIN0207_L6.3mm_D2.5mm_P10.16mm_Horizontal, Resistor_THT:R_Axial_DIN0207_L6.3mm_D2.5mm_P10.16mm_Horizontal, F.Cu at (157.5, 274.3)
- added 1k: R_Axial_DIN0207_L6.3mm_D2.5mm_P10.16mm_Horizontal, Resistor_THT:R_Axial_DIN0207_L6.3mm_D2.5mm_P10.16mm_Horizontal, F.Cu at (137.2, 274.3)
- added 1k: R_Axial_DIN0207_L6.3mm_D2.5mm_P10.16mm_Horizontal, Resistor_THT:R_Axial_DIN0207_L6.3mm_D2.5mm_P10.16mm_Horizontal, F.Cu at (116.8, 274.3)
- added 1k: R_Axial_DIN0207_L6.3mm_D2.5mm_P10.16mm_Horizontal, Resistor_THT:R_Axial_DIN0207_L6.3mm_D2.5mm_P10.16mm_Horizontal, F.Cu at (96.5, 274.3)
- added 1k: R_Axial_DIN0207_L6.3mm_D2.5mm_P10.16mm_Horizontal, Resistor_THT:R_Axial_DIN0207_L6.3mm_D2.5mm_P10.16mm_Horizontal, F.Cu at (76.2, 274.3)
- added 1k: R_Axial_DIN0207_L6.3mm_D2.5mm_P10.16mm_Horizontal, Resistor_THT:R_Axial_DIN0207_L6.3mm_D2.5mm_P10.16mm_Horizontal, F.Cu at (421.6, 254.0)
- added 1k: R_Axial_DIN0207_L6.3mm_D2.5mm_P10.16mm_Horizontal, Resistor_THT:R_Axial_DIN0207_L6.3mm_D2.5mm_P10.16mm_Horizontal, F.Cu at (401.3, 254.0)
- added 1k: R_Axial_DIN0207_L6.3mm_D2.5mm_P10.16mm_Horizontal, Resistor_THT:R_Axial_DIN0207_L6.3mm_D2.5mm_P10.16mm_Horizontal, F.Cu at (381.0, 254.0)
- added 1k: R_Axial_DIN0207_L6.3mm_D2.5mm_P10.16mm_Horizontal, Resistor_THT:R_Axial_DIN0207_L6.3mm_D2.5mm_P10.16mm_Horizontal, F.Cu at (360.7, 254.0)
- added 1k: R_Axial_DIN0207_L6.3mm_D2.5mm_P10.16mm_Horizontal, Resistor_THT:R_Axial_DIN0207_L6.3mm_D2.5mm_P10.16mm_Horizontal, F.Cu at (340.4, 254.0)
- added 1k: R_Axial_DIN0207_L6.3mm_D2.5mm_P10.16mm_Horizontal, Resistor_THT:R_Axial_DIN0207_L6.3mm_D2.5mm_P10.16mm_Horizontal, F.Cu at (320.0, 315.0)
- added 1k: R_Axial_DIN0207_L6.3mm_D2.5mm_P10.16mm_Horizontal, Resistor_THT:R_Axial_DIN0207_L6.3mm_D2.5mm_P10.16mm_Horizontal, F.Cu at (320.0, 254.0)
- added 1k: R_Axial_DIN0207_L6.3mm_D2.5mm_P10.16mm_Horizontal, Resistor_THT:R_Axial_DIN0207_L6.3mm_D2.5mm_P10.16mm_Horizontal, F.Cu at (299.7, 254.0)
- added 1k: R_Axial_DIN0207_L6.3mm_D2.5mm_P10.16mm_Horizontal, Resistor_THT:R_Axial_DIN0207_L6.3mm_D2.5mm_P10.16mm_Horizontal, F.Cu at (279.4, 254.0)
- added 1k: R_Axial_DIN0207_L6.3mm_D2.5mm_P10.16mm_Horizontal, Resistor_THT:R_Axial_DIN0207_L6.3mm_D2.5mm_P10.16mm_Horizontal, F.Cu at (259.1, 254.0)
- added 1k: R_Axial_DIN0207_L6.3mm_D2.5mm_P10.16mm_Horizontal, Resistor_THT:R_Axial_DIN0207_L6.3mm_D2.5mm_P10.16mm_Horizontal, F.Cu at (238.8, 254.0)
- added 1k: R_Axial_DIN0207_L6.3mm_D2.5mm_P10.16mm_Horizontal, Resistor_THT:R_Axial_DIN0207_L6.3mm_D2.5mm_P10.16mm_Horizontal, F.Cu at (218.4, 254.0)
- added 1k: R_Axial_DIN0207_L6.3mm_D2.5mm_P10.16mm_Horizontal, Resistor_THT:R_Axial_DIN0207_L6.3mm_D2.5mm_P10.16mm_Horizontal, F.Cu at (198.1, 254.0)
- added 1k: R_Axial_DIN0207_L6.3mm_D2.5mm_P10.16mm_Horizontal, Resistor_THT:R_Axial_DIN0207_L6.3mm_D2.5mm_P10.16mm_Horizontal, F.Cu at (177.8, 254.0)
- added 1k: R_Axial_DIN0207_L6.3mm_D2.5mm_P10.16mm_Horizontal, Resistor_THT:R_Axial_DIN0207_L6.3mm_D2.5mm_P10.16mm_Horizontal, F.Cu at (157.5, 254.0)
- added 1k: R_Axial_DIN0207_L6.3mm_D2.5mm_P10.16mm_Horizontal, Resistor_THT:R_Axial_DIN0207_L6.3mm_D2.5mm_P10.16mm_Horizontal, F.Cu at (137.2, 254.0)
- added 1k: R_Axial_DIN0207_L6.3mm_D2.5mm_P10.16mm_Horizontal, Resistor_THT:R_Axial_DIN0207_L6.3mm_D2.5mm_P10.16mm_Horizontal, F.Cu at (299.7, 315.0)
- added 1k: R_Axial_DIN0207_L6.3mm_D2.5mm_P10.16mm_Horizontal, Resistor_THT:R_Axial_DIN0207_L6.3mm_D2.5mm_P10.16mm_Horizontal, F.Cu at (116.8, 254.0)
- added 1k: R_Axial_DIN0207_L6.3mm_D2.5mm_P10.16mm_Horizontal, Resistor_THT:R_Axial_DIN0207_L6.3mm_D2.5mm_P10.16mm_Horizontal, F.Cu at (96.5, 254.0)
- added 1k: R_Axial_DIN0207_L6.3mm_D2.5mm_P10.16mm_Horizontal, Resistor_THT:R_Axial_DIN0207_L6.3mm_D2.5mm_P10.16mm_Horizontal, F.Cu at (76.2, 254.0)
- added 1k: R_Axial_DIN0207_L6.3mm_D2.5mm_P10.16mm_Horizontal, Resistor_THT:R_Axial_DIN0207_L6.3mm_D2.5mm_P10.16mm_Horizontal, F.Cu at (421.6, 233.7)
- added 1k: R_Axial_DIN0207_L6.3mm_D2.5mm_P10.16mm_Horizontal, Resistor_THT:R_Axial_DIN0207_L6.3mm_D2.5mm_P10.16mm_Horizontal, F.Cu at (401.3, 233.7)
- added 1k: R_Axial_DIN0207_L6.3mm_D2.5mm_P10.16mm_Horizontal, Resistor_THT:R_Axial_DIN0207_L6.3mm_D2.5mm_P10.16mm_Horizontal, F.Cu at (381.0, 233.7)
- added 1k: R_Axial_DIN0207_L6.3mm_D2.5mm_P10.16mm_Horizontal, Resistor_THT:R_Axial_DIN0207_L6.3mm_D2.5mm_P10.16mm_Horizontal, F.Cu at (360.7, 233.7)
- added 1k: R_Axial_DIN0207_L6.3mm_D2.5mm_P10.16mm_Horizontal, Resistor_THT:R_Axial_DIN0207_L6.3mm_D2.5mm_P10.16mm_Horizontal, F.Cu at (340.4, 233.7)
- added 1k: R_Axial_DIN0207_L6.3mm_D2.5mm_P10.16mm_Horizontal, Resistor_THT:R_Axial_DIN0207_L6.3mm_D2.5mm_P10.16mm_Horizontal, F.Cu at (320.0, 233.7)
- added 1k: R_Axial_DIN0207_L6.3mm_D2.5mm_P10.16mm_Horizontal, Resistor_THT:R_Axial_DIN0207_L6.3mm_D2.5mm_P10.16mm_Horizontal, F.Cu at (299.7, 233.7)
- added 1k: R_Axial_DIN0207_L6.3mm_D2.5mm_P10.16mm_Horizontal, Resistor_THT:R_Axial_DIN0207_L6.3mm_D2.5mm_P10.16mm_Horizontal, F.Cu at (279.4, 315.0)
- added 1k: R_Axial_DIN0207_L6.3mm_D2.5mm_P10.16mm_Horizontal, Resistor_THT:R_Axial_DIN0207_L6.3mm_D2.5mm_P10.16mm_Horizontal, F.Cu at (279.4, 233.7)
- added 1k: R_Axial_DIN0207_L6.3mm_D2.5mm_P10.16mm_Horizontal, Resistor_THT:R_Axial_DIN0207_L6.3mm_D2.5mm_P10.16mm_Horizontal, F.Cu at (259.1, 233.7)
- added 1k: R_Axial_DIN0207_L6.3mm_D2.5mm_P10.16mm_Horizontal, Resistor_THT:R_Axial_DIN0207_L6.3mm_D2.5mm_P10.16mm_Horizontal, F.Cu at (238.8, 233.7)
- added 1k: R_Axial_DIN0207_L6.3mm_D2.5mm_P10.16mm_Horizontal, Resistor_THT:R_Axial_DIN0207_L6.3mm_D2.5mm_P10.16mm_Horizontal, F.Cu at (218.4, 233.7)
- added 1k: R_Axial_DIN0207_L6.3mm_D2.5mm_P10.16mm_Horizontal, Resistor_THT:R_Axial_DIN0207_L6.3mm_D2.5mm_P10.16mm_Horizontal, F.Cu at (198.1, 233.7)
- added 1k: R_Axial_DIN0207_L6.3mm_D2.5mm_P10.16mm_Horizontal, Resistor_THT:R_Axial_DIN0207_L6.3mm_D2.5mm_P10.16mm_Horizontal, F.Cu at (177.8, 233.7)
- added 1k: R_Axial_DIN0207_L6.3mm_D2.5mm_P10.16mm_Horizontal, Resistor_THT:R_Axial_DIN0207_L6.3mm_D2.5mm_P10.16mm_Horizontal, F.Cu at (157.5, 233.7)
- added 1k: R_Axial_DIN0207_L6.3mm_D2.5mm_P10.16mm_Horizontal, Resistor_THT:R_Axial_DIN0207_L6.3mm_D2.5mm_P10.16mm_Horizontal, F.Cu at (137.2, 233.7)
- added 1k: R_Axial_DIN0207_L6.3mm_D2.5mm_P10.16mm_Horizontal, Resistor_THT:R_Axial_DIN0207_L6.3mm_D2.5mm_P10.16mm_Horizontal, F.Cu at (116.8, 233.7)
- added 1k: R_Axial_DIN0207_L6.3mm_D2.5mm_P10.16mm_Horizontal, Resistor_THT:R_Axial_DIN0207_L6.3mm_D2.5mm_P10.16mm_Horizontal, F.Cu at (96.5, 233.7)
- added 1k: R_Axial_DIN0207_L6.3mm_D2.5mm_P10.16mm_Horizontal, Resistor_THT:R_Axial_DIN0207_L6.3mm_D2.5mm_P10.16mm_Horizontal, F.Cu at (259.1, 315.0)
- added 1k: R_Axial_DIN0207_L6.3mm_D2.5mm_P10.16mm_Horizontal, Resistor_THT:R_Axial_DIN0207_L6.3mm_D2.5mm_P10.16mm_Horizontal, F.Cu at (76.2, 233.7)
- added 1k: R_Axial_DIN0207_L6.3mm_D2.5mm_P10.16mm_Horizontal, Resistor_THT:R_Axial_DIN0207_L6.3mm_D2.5mm_P10.16mm_Horizontal, F.Cu at (421.6, 213.4)
- added 1k: R_Axial_DIN0207_L6.3mm_D2.5mm_P10.16mm_Horizontal, Resistor_THT:R_Axial_DIN0207_L6.3mm_D2.5mm_P10.16mm_Horizontal, F.Cu at (401.3, 213.4)
- added 1k: R_Axial_DIN0207_L6.3mm_D2.5mm_P10.16mm_Horizontal, Resistor_THT:R_Axial_DIN0207_L6.3mm_D2.5mm_P10.16mm_Horizontal, F.Cu at (381.0, 213.4)
- added 1k: R_Axial_DIN0207_L6.3mm_D2.5mm_P10.16mm_Horizontal, Resistor_THT:R_Axial_DIN0207_L6.3mm_D2.5mm_P10.16mm_Horizontal, F.Cu at (360.7, 213.4)
- added 1k: R_Axial_DIN0207_L6.3mm_D2.5mm_P10.16mm_Horizontal, Resistor_THT:R_Axial_DIN0207_L6.3mm_D2.5mm_P10.16mm_Horizontal, F.Cu at (340.4, 213.4)
- added 1k: R_Axial_DIN0207_L6.3mm_D2.5mm_P10.16mm_Horizontal, Resistor_THT:R_Axial_DIN0207_L6.3mm_D2.5mm_P10.16mm_Horizontal, F.Cu at (320.0, 213.4)
- added 1k: R_Axial_DIN0207_L6.3mm_D2.5mm_P10.16mm_Horizontal, Resistor_THT:R_Axial_DIN0207_L6.3mm_D2.5mm_P10.16mm_Horizontal, F.Cu at (299.7, 213.4)
- added 1k: R_Axial_DIN0207_L6.3mm_D2.5mm_P10.16mm_Horizontal, Resistor_THT:R_Axial_DIN0207_L6.3mm_D2.5mm_P10.16mm_Horizontal, F.Cu at (279.4, 213.4)
- added 1k: R_Axial_DIN0207_L6.3mm_D2.5mm_P10.16mm_Horizontal, Resistor_THT:R_Axial_DIN0207_L6.3mm_D2.5mm_P10.16mm_Horizontal, F.Cu at (259.1, 213.4)
- added GND: TestPoint_Plated_Hole_D2.0mm, TestPoint:TestPoint_Plated_Hole_D2.0mm, F.Cu at (55.9, 203.2)
- added REF**: LED_D5.0mm, LED_THT:LED_D5.0mm, F.Cu at (426.7, 309.9)
- added REF**: LED_D5.0mm, LED_THT:LED_D5.0mm, F.Cu at (243.8, 309.9)
- added REF**: LED_D5.0mm, LED_THT:LED_D5.0mm, F.Cu at (243.8, 208.3)
- added REF**: LED_D5.0mm, LED_THT:LED_D5.0mm, F.Cu at (223.5, 208.3)
- added REF**: LED_D5.0mm, LED_THT:LED_D5.0mm, F.Cu at (203.2, 208.3)
- added REF**: LED_D5.0mm, LED_THT:LED_D5.0mm, F.Cu at (182.9, 208.3)
- added REF**: LED_D5.0mm, LED_THT:LED_D5.0mm, F.Cu at (162.6, 208.3)
- added REF**: LED_D5.0mm, LED_THT:LED_D5.0mm, F.Cu at (142.2, 208.3)
- added REF**: LED_D5.0mm, LED_THT:LED_D5.0mm, F.Cu at (121.9, 208.3)
- added REF**: LED_D5.0mm, LED_THT:LED_D5.0mm, F.Cu at (101.6, 208.3)
- added REF**: LED_D5.0mm, LED_THT:LED_D5.0mm, F.Cu at (81.3, 208.3)
- added REF**: LED_D5.0mm, LED_THT:LED_D5.0mm, F.Cu at (426.7, 188.0)
- added REF**: LED_D5.0mm, LED_THT:LED_D5.0mm, F.Cu at (223.5, 309.9)
- added REF**: LED_D5.0mm, LED_THT:LED_D5.0mm, F.Cu at (406.4, 188.0)
- added REF**: LED_D5.0mm, LED_THT:LED_D5.0mm, F.Cu at (386.1, 188.0)
- added REF**: LED_D5.0mm, LED_THT:LED_D5.0mm, F.Cu at (365.8, 188.0)
- added REF**: LED_D5.0mm, LED_THT:LED_D5.0mm, F.Cu at (345.4, 188.0)
- added REF**: LED_D5.0mm, LED_THT:LED_D5.0mm, F.Cu at (325.1, 188.0)
- added REF**: LED_D5.0mm, LED_THT:LED_D5.0mm, F.Cu at (304.8, 188.0)
- added REF**: LED_D5.0mm, LED_THT:LED_D5.0mm, F.Cu at (284.5, 188.0)
- added REF**: LED_D5.0mm, LED_THT:LED_D5.0mm, F.Cu at (264.2, 188.0)
- added REF**: LED_D5.0mm, LED_THT:LED_D5.0mm, F.Cu at (243.8, 188.0)
- added REF**: LED_D5.0mm, LED_THT:LED_D5.0mm, F.Cu at (223.5, 188.0)
- added REF**: LED_D5.0mm, LED_THT:LED_D5.0mm, F.Cu at (203.2, 309.9)
- added REF**: LED_D5.0mm, LED_THT:LED_D5.0mm, F.Cu at (203.2, 188.0)
- added REF**: LED_D5.0mm, LED_THT:LED_D5.0mm, F.Cu at (182.9, 188.0)
- added REF**: LED_D5.0mm, LED_THT:LED_D5.0mm, F.Cu at (162.6, 188.0)
- added REF**: LED_D5.0mm, LED_THT:LED_D5.0mm, F.Cu at (142.2, 188.0)
- added REF**: LED_D5.0mm, LED_THT:LED_D5.0mm, F.Cu at (121.9, 188.0)
- added REF**: LED_D5.0mm, LED_THT:LED_D5.0mm, F.Cu at (101.6, 188.0)
- added REF**: LED_D5.0mm, LED_THT:LED_D5.0mm, F.Cu at (81.3, 188.0)
- added REF**: LED_D5.0mm, LED_THT:LED_D5.0mm, F.Cu at (426.7, 167.6)
- added REF**: LED_D5.0mm, LED_THT:LED_D5.0mm, F.Cu at (406.4, 167.6)
- added REF**: LED_D5.0mm, LED_THT:LED_D5.0mm, F.Cu at (386.1, 167.6)
- added REF**: LED_D5.0mm, LED_THT:LED_D5.0mm, F.Cu at (182.9, 309.9)
- added REF**: LED_D5.0mm, LED_THT:LED_D5.0mm, F.Cu at (365.8, 167.6)
- added REF**: LED_D5.0mm, LED_THT:LED_D5.0mm, F.Cu at (345.4, 167.6)
- added REF**: LED_D5.0mm, LED_THT:LED_D5.0mm, F.Cu at (325.1, 167.6)
- added REF**: LED_D5.0mm, LED_THT:LED_D5.0mm, F.Cu at (304.8, 167.6)
- added REF**: LED_D5.0mm, LED_THT:LED_D5.0mm, F.Cu at (284.5, 167.6)
- added REF**: LED_D5.0mm, LED_THT:LED_D5.0mm, F.Cu at (264.2, 167.6)
- added REF**: LED_D5.0mm, LED_THT:LED_D5.0mm, F.Cu at (243.8, 167.6)
- added REF**: LED_D5.0mm, LED_THT:LED_D5.0mm, F.Cu at (223.5, 167.6)
- added REF**: LED_D5.0mm, LED_THT:LED_D5.0mm, F.Cu at (203.2, 167.6)
- added REF**: LED_D5.0mm, LED_THT:LED_D5.0mm, F.Cu at (182.9, 167.6)
- added REF**: LED_D5.0mm, LED_THT:LED_D5.0mm, F.Cu at (162.6, 309.9)
- added REF**: LED_D5.0mm, LED_THT:LED_D5.0mm, F.Cu at (162.6, 167.6)
- added REF**: LED_D5.0mm, LED_THT:LED_D5.0mm, F.Cu at (142.2, 167.6)
- added REF**: LED_D5.0mm, LED_THT:LED_D5.0mm, F.Cu at (121.9, 167.6)
- added REF**: LED_D5.0mm, LED_THT:LED_D5.0mm, F.Cu at (101.6, 167.6)
- added REF**: LED_D5.0mm, LED_THT:LED_D5.0mm, F.Cu at (81.3, 167.6)
- added REF**: LED_D5.0mm, LED_THT:LED_D5.0mm, F.Cu at (426.7, 147.3)
- added REF**: LED_D5.0mm, LED_THT:LED_D5.0mm, F.Cu at (406.4, 147.3)
- added REF**: LED_D5.0mm, LED_THT:LED_D5.0mm, F.Cu at (386.1, 147.3)
- added REF**: LED_D5.0mm, LED_THT:LED_D5.0mm, F.Cu at (365.8, 147.3)
- added REF**: LED_D5.0mm, LED_THT:LED_D5.0mm, F.Cu at (345.4, 147.3)
- added REF**: LED_D5.0mm, LED_THT:LED_D5.0mm, F.Cu at (142.2, 309.9)
- added REF**: LED_D5.0mm, LED_THT:LED_D5.0mm, F.Cu at (325.1, 147.3)
- added REF**: LED_D5.0mm, LED_THT:LED_D5.0mm, F.Cu at (304.8, 147.3)
- added REF**: LED_D5.0mm, LED_THT:LED_D5.0mm, F.Cu at (284.5, 147.3)
- added REF**: LED_D5.0mm, LED_THT:LED_D5.0mm, F.Cu at (264.2, 147.3)
- added REF**: LED_D5.0mm, LED_THT:LED_D5.0mm, F.Cu at (243.8, 147.3)
- added REF**: LED_D5.0mm, LED_THT:LED_D5.0mm, F.Cu at (223.5, 147.3)
- added REF**: LED_D5.0mm, LED_THT:LED_D5.0mm, F.Cu at (203.2, 147.3)
- added REF**: LED_D5.0mm, LED_THT:LED_D5.0mm, F.Cu at (182.9, 147.3)
- added REF**: LED_D5.0mm, LED_THT:LED_D5.0mm, F.Cu at (162.6, 147.3)
- added REF**: LED_D5.0mm, LED_THT:LED_D5.0mm, F.Cu at (142.2, 147.3)
- added REF**: LED_D5.0mm, LED_THT:LED_D5.0mm, F.Cu at (121.9, 309.9)
- added REF**: LED_D5.0mm, LED_THT:LED_D5.0mm, F.Cu at (121.9, 147.3)
- added REF**: LED_D5.0mm, LED_THT:LED_D5.0mm, F.Cu at (101.6, 147.3)
- added REF**: LED_D5.0mm, LED_THT:LED_D5.0mm, F.Cu at (81.3, 147.3)
- added REF**: LED_D5.0mm, LED_THT:LED_D5.0mm, F.Cu at (426.7, 127.0)
- added REF**: LED_D5.0mm, LED_THT:LED_D5.0mm, F.Cu at (406.4, 127.0)
- added REF**: LED_D5.0mm, LED_THT:LED_D5.0mm, F.Cu at (386.1, 127.0)
- added REF**: LED_D5.0mm, LED_THT:LED_D5.0mm, F.Cu at (365.8, 127.0)
- added REF**: LED_D5.0mm, LED_THT:LED_D5.0mm, F.Cu at (345.4, 127.0)
- added REF**: LED_D5.0mm, LED_THT:LED_D5.0mm, F.Cu at (325.1, 127.0)
- added REF**: LED_D5.0mm, LED_THT:LED_D5.0mm, F.Cu at (304.8, 127.0)
- added REF**: LED_D5.0mm, LED_THT:LED_D5.0mm, F.Cu at (101.6, 309.9)
- added REF**: LED_D5.0mm, LED_THT:LED_D5.0mm, F.Cu at (284.5, 127.0)
- added REF**: LED_D5.0mm, LED_THT:LED_D5.0mm, F.Cu at (264.2, 127.0)
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Routing:
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Other:
- board outline added: 420 x 297 mm
- board text added: "A3-led-panel v1 2020-07-18 OSH CC-0"
